File: PCB/MacroPadv1-HackClub.kicad_sch (KiCad schematic)
At the start: 33 parts, among them SW1 SW_Push, SW10 SW_Push, SW11 SW_Push, SW12 SW_Push, SW13 SW_Push, SW14 SW_Push, SW15 SW_Push, SW16 SW_Push, SW2 SW_Push, SW3 SW_Push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

Commit message: Pcb rerouting
Parts:
- D1, D10, D11, D12, D13, D14, D15, D16, D2, D3, D4, D5, D6, D7, D8, D9: value SK6812MINI -> SK6812MINI-E; footprint LED_SMD:LED_SK6812MINI_PLCC4_3.5x3.5mm_P1.75mm -> kicad-keyboard-parts.pretty-master:MX_SK6812MINI-E
Changed lines of the file:
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@@
 			)
 		)
-		(property "Value" "SK6812MINI"
+		(property "Value" "SK6812MINI-E"
 			(at 107.95 27.8698 0)
 			(effects
@@
 			)
 		)
-		(property "Footprint" "LED_SMD:LED_SK6812MINI_PLCC4_3.5x3.5mm_P1.75mm"
+		(property "Footprint" "kicad-keyboard-parts.pretty-master:MX_SK6812MINI-E"
 			(at 96.52 39.37 0)
 			(effects
@@
 			)
 		)
-		(property "Value" "SK6812MINI"
+		(property "Value" "SK6812MINI-E"
 			(at 52.07 48.1898 0)
 			(effects
@@
 			)
 		)
-		(property "Footprint" "LED_SMD:LED_SK6812MINI_PLCC4_3.5x3.5mm_P1.75mm"
+		(property "Footprint" "kicad-keyboard-parts.pretty-master:MX_SK6812MINI-E"
 			(at 40.64 59.69 0)
 			(effects
@@
 			)
 		)
-		(property "Value" "SK6812MINI"
+		(property "Value" "SK6812MINI-E"
 			(at 142.24 48.1898 0)
 			(effects
@@
 			)
 		)
-		(property "Footprint" "LED_SMD:LED_SK6812MINI_PLCC4_3.5x3.5mm_P1.75mm"
+		(property "Footprint" "kicad-keyboard-parts.pretty-master:MX_SK6812MINI-E"
 			(at 130.81 59.69 0)
 			(effects
@@
 			)
 		)
-		(property "Value" "SK6812MINI"
+		(property "Value" "SK6812MINI-E"
 			(at 77.47 48.1898 0)
 			(effects
@@
 			)
 		)
-		(property "Footprint" "LED_SMD:LED_SK6812MINI_PLCC4_3.5x3.5mm_P1.75mm"
+		(property "Footprint" "kicad-keyboard-parts.pretty-master:MX_SK6812MINI-E"
 			(at 66.04 59.69 0)
 			(effects
@@
 			)
 		)
-		(property "Value" "SK6812MINI"
+		(property "Value" "SK6812MINI-E"
 			(at 52.07 27.8698 0)
 			(effects
@@
 			)
 		)
-		(property "Footprint" "LED_SMD:LED_SK6812MINI_PLCC4_3.5x3.5mm_P1.75mm"
+		(property "Footprint" "kicad-keyboard-parts.pretty-master:MX_SK6812MINI-E"
 			(at 40.64 39.37 0)
 			(effects
@@
 			)
 		)
-		(property "Value" "SK6812MINI"
+		(property "Value" "SK6812MINI-E"
 			(at 171.45 29.1398 0)
 			(effects
@@
 			)
 		)
-		(property "Footprint" "LED_SMD:LED_SK6812MINI_PLCC4_3.5x3.5mm_P1.75mm"
+		(property "Footprint" "kicad-keyboard-parts.pretty-master:MX_SK6812MINI-E"
 			(at 160.02 40.64 0)
 			(effects
@@
 			)
 		)
-		(property "Value" "SK6812MINI"
+		(property "Value" "SK6812MINI-E"
 			(at 109.22 48.1898 0)
 			(effects
@@
 			)
 		)
-		(property "Footprint" "LED_SMD:LED_SK6812MINI_PLCC4_3.5x3.5mm_P1.75mm"
+		(property "Footprint" "kicad-keyboard-parts.pretty-master:MX_SK6812MINI-E"
 			(at 97.79 59.69 0)
 			(effects
@@
 			)
 		)
-		(property "Value" "SK6812MINI"
+		(property "Value" "SK6812MINI-E"
 			(at 267.97 26.5998 0)
 			(effects
@@
 			)
 		)
-		(property "Footprint" "LED_SMD:LED_SK6812MINI_PLCC4_3.5x3.5mm_P1.75mm"
+		(property "Footprint" "kicad-keyboard-parts.pretty-master:MX_SK6812MINI-E"
 			(at 256.54 38.1 0)
 			(effects
@@
 			)
 		)
-		(property "Value" "SK6812MINI"
+		(property "Value" "SK6812MINI-E"
 			(at 78.74 27.8698 0)
 			(effects
@@
 			)
 		)
-		(property "Footprint" "LED_SMD:LED_SK6812MINI_PLCC4_3.5x3.5mm_P1.75mm"
+		(property "Footprint" "kicad-keyboard-parts.pretty-master:MX_SK6812MINI-E"
 			(at 67.31 39.37 0)
 			(effects
@@
 			)
 		)
-		(property "Value" "SK6812MINI"
+		(property "Value" "SK6812MINI-E"
 			(at 203.2 27.8698 0)
 			(effects
@@
 			)
 		)
-		(property "Footprint" "LED_SMD:LED_SK6812MINI_PLCC4_3.5x3.5mm_P1.75mm"
+		(property "Footprint" "kicad-keyboard-parts.pretty-master:MX_SK6812MINI-E"
 			(at 191.77 39.37 0)
 			(effects
@@
 			)
 		)
-		(property "Value" "SK6812MINI"
+		(property "Value" "SK6812MINI-E"
 			(at 171.45 46.9198 0)
 			(effects
@@
 			)
 		)
-		(property "Footprint" "LED_SMD:LED_SK6812MINI_PLCC4_3.5x3.5mm_P1.75mm"
+		(property "Footprint" "kicad-keyboard-parts.pretty-master:MX_SK6812MINI-E"
 			(at 160.02 58.42 0)
 			(effects
@@
 			)
 		)
-		(property "Value" "SK6812MINI"
+		(property "Value" "SK6812MINI-E"
 			(at 142.24 27.8698 0)
 			(effects
@@
 			)
 		)
-		(property "Footprint" "LED_SMD:LED_SK6812MINI_PLCC4_3.5x3.5mm_P1.75mm"
+		(property "Footprint" "kicad-keyboard-parts.pretty-master:MX_SK6812MINI-E"
 			(at 130.81 39.37 0)
 			(effects
@@
 			)
 		)
-		(property "Value" "SK6812MINI"
+		(property "Value" "SK6812MINI-E"
 			(at 201.93 45.6498 0)
 			(effects
@@
 			)
 		)
-		(property "Footprint" "LED_SMD:LED_SK6812MINI_PLCC4_3.5x3.5mm_P1.75mm"
+		(property "Footprint" "kicad-keyboard-parts.pretty-master:MX_SK6812MINI-E"
 			(at 190.5 57.15 0)
 			(effects
@@
 			)
 		)
-		(property "Value" "SK6812MINI"
+		(property "Value" "SK6812MINI-E"
 			(at 236.22 46.9198 0)
 			(effects
@@
 			)
 		)
-		(property "Footprint" "LED_SMD:LED_SK6812MINI_PLCC4_3.5x3.5mm_P1.75mm"
+		(property "Footprint" "kicad-keyboard-parts.pretty-master:MX_SK6812MINI-E"
 			(at 224.79 58.42 0)
 			(effects
@@
 			)
 		)
-		(property "Value" "SK6812MINI"
+		(property "Value" "SK6812MINI-E"
 			(at 269.24 45.6498 0)
 			(effects
@@
 			)
 		)
-		(property "Footprint" "LED_SMD:LED_SK6812MINI_PLCC4_3.5x3.5mm_P1.75mm"
+		(property "Footprint" "kicad-keyboard-parts.pretty-master:MX_SK6812MINI-E"
 			(at 257.81 57.15 0)
 			(effects
@@
 			)
 		)
-		(property "Value" "SK6812MINI"
+		(property "Value" "SK6812MINI-E"
 			(at 236.22 27.8698 0)
 			(effects
@@
 			)
 		)
-		(property "Footprint" "LED_SMD:LED_SK6812MINI_PLCC4_3.5x3.5mm_P1.75mm"
+		(property "Footprint" "kicad-keyboard-parts.pretty-master:MX_SK6812MINI-E"
 			(at 224.79 39.37 0)
 			(effects
